File: pcb/BTTF-Plutonium.kicad_sch (KiCad schematic)
At the start: 41 parts, among them J1 ESP32 JTAG, J2 ESP32 Prog, J3 Conn_01x03_Pin, J4 Barrel_Jack_Switch, J5 Conn_01x03_Pin, J6 Conn_01x03_Pin, Q1 PMOS, SW1 SW_Push, SW2 SW_Push, U1 BQ21040DBVR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

Commit message: Tidy up plutonium
Parts:
- J4: now not fitted; now left out of the parts list
Changed lines of the file:
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@@
   )
   (symbol (lib_id "Connector:Barrel_Jack_Switch") (at 287.02 33.02 0) (unit 1)
-    (in_bom yes) (on_board yes) (dnp no) (fields_autoplaced)
+    (in_bom no) (on_board no) (dnp yes) (fields_autoplaced)
     (property "Reference" "J4" (at 287.02 25.4 0)
       (effects (font (size 1.27 1.27)))
@@
       (effects (font (size 1.27 1.27)) hide)
     )
+    (property "Sim.Enable" "0" (at 287.02 33.02 0)
+      (effects (font (size 1.27 1.27)) hide)
+    )

Commit message: Moving bits around
Parts:
- added Q2: PMOS, Package_SO:SSOP-8_3.9x5.05mm_P1.27mm, symbol Simulation_SPICE:PMOS
- added R9: 100k, Resistor_SMD:R_0603_1608Metric, symbol Device:R_Small
Connections:
- net +BATT: now also Q2.5 (D), Q2.6 (D), Q2.7 (D), Q2.8 (D)
- net GND: now also R9.2
- net VCC: now also Q2.1 (S), Q2.2 (S), Q2.3 (S); no longer J5.1 (Pin_1), Q1.1 (S), Q1.2 (S), Q1.3 (S)
- net VDD: now also Q2.4 (G), R9.1
- new net VD: J5.1 (Pin_1), Q1.1 (S), Q1.2 (S), Q1.3 (S)
Other:
- note removed: "SMALLER BUTTONS"
