File: pcb/BTTF-Plutonium.kicad_pcb (KiCad board)
At the start: 4 copper layers, 42 x 42 mm, 41 parts, among them J1 ESP32 JTAG, J2 ESP32 Prog, J3 Conn_01x03_Pin, J5 Conn_01x03_Pin, J6 Conn_01x03_Pin, Q1 PMOS, SW1 SW_Push, SW2 SW_Push, U1 BQ21040DBVR, U2 MAX17048G+T10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

Commit message: Tidy up plutonium
Routing:
- net +BATT: track 35.9 -> 29.0 mm
- net ESP_LED_DATA: track 27.1 -> 22.1 mm
- net VCC: track 31.8 -> 30.4 mm
- net ESP32_I2C_SDA: track 36.1 -> 36.7 mm
- net VDD: vias 2 -> 4
- added copper zone on B.Cu, net VDD
- added copper zone on F.Cu, net VDD
Other:
- board text added: "+ TS GND Battery"
- board text added: "ESP32"
- board text added: "GND DATA + LED"

Commit message: Moving bits around
Parts:
- added Q2: PMOS, Package_SO:SSOP-8_3.9x5.05mm_P1.27mm, F.Cu at (144.1, 103.9)
- added R9: 100k, Resistor_SMD:R_0603_1608Metric, F.Cu at (142.2, 107.5)
- moved R1 1.78 mm to (136.9, 92.1)
Connections:
- J5 pad 1: VCC -> VD
- Q1 pad 1: VCC -> VD
- Q1 pad 2: VCC -> VD
- Q1 pad 3: VCC -> VD
Routing:
- net ESP_EN: track 35.3 -> 20.4 mm
- net VDD: track 44.5 -> 58.0 mm, vias 4 -> 5
- net +BATT: track 29.0 -> 41.4 mm, vias 2 -> 0
- net VCC: track 30.4 -> 23.3 mm
- net ESP32_I2C_SCL: track 31.0 -> 35.1 mm
- net BATT_TS: track 15.8 -> 19.5 mm, vias 0 -> 1
- net GND: track 52.0 -> 53.3 mm, vias 34 -> 35
- net ESP32_I2C_SDA: track 36.7 -> 36.8 mm, vias 2 -> 1
- added copper zone on F.Cu, net VD

Commit message: Blank slate
Parts:
- moved U4 63.8 mm to (97.0, 53.9)
- moved R1 63.7 mm to (82.8, 58.5)
- moved R4 56.4 mm to (83.6, 61.8)
- moved C3 44.2 mm to (121.8, 59.9)
- moved R2 44.2 mm to (119.6, 63.0)
- moved C1 44.2 mm to (120.5, 59.9)
- moved D1 44.2 mm to (113.8, 62.0)
- moved U1 44.2 mm to (117.6, 60.4)
- moved C4 44.2 mm to (117.5, 56.5)
- moved C5 44.2 mm to (117.5, 57.8)
- moved R3 44.2 mm to (113.8, 60.5)
- moved Q2 39.9 mm to (178.5, 124.1)
- moved R9 39.9 mm to (176.6, 127.7)
- moved C11 34.4 mm to (108.3, 131.7)
- moved C12 34.4 mm to (106.9, 131.7)
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Routing:
- net VDD: track 58.0 -> 0.00 mm, vias 5 -> 0
- net GND: track 53.3 -> 0.00 mm, vias 35 -> 0
- net ESP_IO0: track 46.8 -> 0.00 mm, vias 2 -> 0
- net +BATT: track 41.4 -> 0.00 mm
- net ESP32_I2C_SDA: track 36.8 -> 0.00 mm, vias 1 -> 0
- net ESP_CONNECTION_BUTTON: track 36.1 -> 0.00 mm, vias 1 -> 0
- net ESP32_I2C_SCL: track 35.1 -> 0.00 mm, vias 1 -> 0
- net VCC: track 23.3 -> 0.00 mm
- net ESP_LED_DATA: track 22.1 -> 0.00 mm
- net ESP_EN: track 20.4 -> 0.00 mm, vias 2 -> 0
- net BATT_TS: track 19.5 -> 0.00 mm, vias 1 -> 0
- net +3.3V: track 17.0 -> 0.00 mm, vias 12 -> 0
- net ESP_TDO: track 10.1 -> 0.00 mm
- net ESP_UART_RX: track 9.06 -> 0.00 mm
- net ESP_TDI: track 9.00 -> 0.00 mm
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- removed copper zone on F.Cu, net +3.3V
- removed copper zone on F.Cu, net +BATT
- removed copper zone on F.Cu, net /BATT_FUSE
- removed copper zone on F.Cu, net VCC
- removed copper zone on F.Cu, net VD
- removed copper zone on B.Cu, net VDD
- removed copper zone on F.Cu, net VDD
Other:
- board text removed: "ESP32"

Commit message: Part placement
Parts:
- SW1, SW2: moved to B.Cu
- moved R1 81.2 mm to (156.6, 92.4), turned to 90 degrees
- moved R4 80.2 mm to (157.7, 92.4), turned to 90 degrees
- moved U4 65.9 mm to (140.1, 103.8), turned to -90 degrees
- moved C1 49.1 mm to (153.5, 96.2)
- moved C4 49.1 mm to (150.5, 92.8)
- moved C5 49.1 mm to (150.5, 94.2)
- moved R2 49.1 mm to (152.6, 99.3)
- moved C3 49.1 mm to (154.8, 96.2)
- moved D1 49.1 mm to (146.8, 98.5)
- moved U1 49.1 mm to (150.5, 96.8)
- moved R3 49.1 mm to (146.8, 96.8)
- moved Q2 47.2 mm to (140.8, 95.7), turned to 90 degrees
- moved R6 47.2 mm to (159.7, 98.0), turned to -90 degrees
- moved C12 45.5 mm to (132.6, 94.2), turned to 0 degrees
- moved R5 45.2 mm to (159.6, 101.8), turned to 90 degrees
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Routing:
- net VDD: track 0.00 -> 58.7 mm
- net ESP_IO0: track 0.00 -> 32.1 mm, vias 0 -> 1
- net BATT_TS: track 0.00 -> 31.1 mm
- net +BATT: track 0.00 -> 26.0 mm
- net GND: track 0.00 -> 21.1 mm, vias 0 -> 20
- net VCC: track 0.00 -> 11.3 mm
- net ESP_UART_RX: track 0.00 -> 11.1 mm
- net ESP_UART_TX: track 0.00 -> 9.25 mm
- net +3.3V: track 0.00 -> 8.60 mm, vias 0 -> 4
- net /VBUS: track 0.00 -> 7.22 mm
- net ESP_TDO: track 0.00 -> 6.61 mm
- net ESP_TDI: track 0.00 -> 5.57 mm
- net ESP_TMS: track 0.00 -> 4.30 mm
- net ESP_TCK: track 0.00 -> 4.19 mm
- net ESP32_I2C_SDA: track 0.00 -> 4.17 mm
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- added copper zone on F.Cu, net +BATT
- added copper zone on F.Cu, net /BATT_FUSE
- added copper zone on F.Cu, net VCC
- added copper zone on F.Cu, net VD

Commit message: Routing complete, new switch needed
Parts:
- moved C10 0.29 mm to (134.6, 108.9)
- moved C9 0.29 mm to (134.6, 110.2)
Routing:
- net ESP_EN: track 2.27 -> 49.5 mm, vias 1 -> 2
- net GND: track 21.1 -> 44.8 mm, vias 20 -> 33
- net ESP_CONNECTION_BUTTON: track 0.00 -> 18.2 mm, vias 0 -> 1
- net ESP_IO0: track 32.1 -> 50.1 mm
- net ESP_LED_DATA: track 0.00 -> 14.9 mm
- net ESP32_I2C_SDA: track 4.17 -> 18.0 mm, vias 0 -> 1
- net ESP32_I2C_SCL: track 2.80 -> 16.2 mm, vias 0 -> 1
- net BATT_TS: track 31.1 -> 35.6 mm
- net VCC: track 11.3 -> 15.1 mm
- net +3.3V: track 8.60 -> 12.0 mm, vias 4 -> 11
- added copper zone on F.Cu, net +3.3V
Other:
- board text added: "+ GND -> CHARGER"
